File: Initial Schematic.sch (EAGLE design)
At the start: 9 parts, among them J1 CONNECTOR, U1 CAN_TRANSCAN_TRANS

Commit message: Layout v3
Parts:
- added C1: 1uF, NFR23:CAPACITORC1206
- added R5: 120, NFR23:RESISTORR1206
- R1, R2: device NFR23:RESISTORR0603 -> NFR23:RESISTORR1206
- R3: value 1k -> 2k; device NFR23:RESISTORR0603 -> NFR23:RESISTORR1206
- R4: value 2k -> 1k; device NFR23:RESISTORR0603 -> NFR23:RESISTORR1206
Connections:
- new net EN: C1.2, U$1.EN
- net BRAKE_3V3: now also R3.2, R4.1; no longer R3.1, R4.2
- net BRAKE_5V: now also R4.2; no longer R3.2
- net CANH: now also R5.1
- net CANL: now also R5.2
- net GND: now also C1.1, R3.1; no longer R4.1
Other:
- moved on the sheet: R3, R4
Changed lines of the file:
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@@
 <part name="U1" library="NFR23" deviceset="CAN_TRANS" device="CAN_TRANS"/>
 <part name="LD1" library="led" library_urn="urn:adsk.eagle:library:259" deviceset="PL006*" device="-WCR21" package3d_urn="urn:adsk.eagle:package:28738/2"/>
-<part name="R1" library="NFR23" deviceset="RESISTOR" device="R0603" package3d_urn="urn:adsk.eagle:package:23555/3" value="330"/>
 <part name="LD2" library="led" library_urn="urn:adsk.eagle:library:259" deviceset="PL006*" device="-WCR21" package3d_urn="urn:adsk.eagle:package:28738/2"/>
-<part name="R2" library="NFR23" deviceset="RESISTOR" device="R0603" package3d_urn="urn:adsk.eagle:package:23555/3" value="330"/>
-<part name="R3" library="NFR23" deviceset="RESISTOR" device="R0603" package3d_urn="urn:adsk.eagle:package:23555/3" value="1k"/>
-<part name="R4" library="NFR23" deviceset="RESISTOR" device="R0603" package3d_urn="urn:adsk.eagle:package:23555/3" value="2k"/>
+<part name="R2" library="NFR23" deviceset="RESISTOR" device="R1206" package3d_urn="urn:adsk.eagle:package:23540/2" value="330"/>
+<part name="R1" library="NFR23" deviceset="RESISTOR" device="R1206" package3d_urn="urn:adsk.eagle:package:23540/2" value="330"/>
+<part name="R3" library="NFR23" deviceset="RESISTOR" device="R1206" package3d_urn="urn:adsk.eagle:package:23540/2" value="2k"/>
+<part name="R4" library="NFR23" deviceset="RESISTOR" device="R1206" package3d_urn="urn:adsk.eagle:package:23540/2" value="1k"/>
+<part name="R5" library="NFR23" deviceset="RESISTOR" device="R1206" package3d_urn="urn:adsk.eagle:package:23540/2" value="120"/>
+<part name="C1" library="NFR23" deviceset="CAPACITOR" device="C1206" package3d_urn="urn:adsk.eagle:package:23618/2" value="1uF"/>
 </parts>
 <sheets>
@@
 <attribute name="NAME" x="-10.668" y="1.016" size="1.778" layer="95" rot="R180"/>
 </instance>
+<instance part="LD2" gate="G$1" x="-27.94" y="33.02" smashed="yes" rot="MR90">
+<attribute name="NAME" x="-32.512" y="36.576" size="1.778" layer="95" rot="MR180"/>
+</instance>
+<instance part="R2" gate="G$1" x="-40.64" y="33.02" smashed="yes">
+<attribute name="NAME" x="-44.45" y="34.5186" size="1.778" layer="95"/>
+<attribute name="VALUE" x="-44.45" y="29.718" size="1.778" layer="96"/>
+</instance>
 <instance part="R1" gate="G$1" x="-25.4" y="-2.54" smashed="yes">
 <attribute name="NAME" x="-29.21" y="-1.0414" size="1.778" layer="95"/>
 <attribute name="VALUE" x="-29.21" y="-5.842" size="1.778" layer="96"/>
 </instance>
-<instance part="LD2" gate="G$1" x="-27.94" y="33.02" smashed="yes" rot="MR90">
-<attribute name="NAME" x="-32.512" y="36.576" size="1.778" layer="95" rot="MR180"/>
-</instance>
-<instance part="R2" gate="G$1" x="-40.64" y="33.02" smashed="yes">
-<attribute name="NAME" x="-44.45" y="34.5186" size="1.778" layer="95"/>
-<attribute name="VALUE" x="-44.45" y="29.718" size="1.778" layer="96"/>
-</instance>
-<instance part="R3" gate="G$1" x="88.9" y="10.16" smashed="yes">
+<instance part="R3" gate="G$1" x="71.12" y="10.16" smashed="yes">
+<attribute name="NAME" x="67.31" y="11.6586" size="1.778" layer="95"/>
+<attribute name="VALUE" x="67.31" y="6.858" size="1.778" layer="96"/>
+</instance>
+<instance part="R4" gate="G$1" x="88.9" y="10.16" smashed="yes">
 <attribute name="NAME" x="85.09" y="11.6586" size="1.778" layer="95"/>
 <attribute name="VALUE" x="85.09" y="6.858" size="1.778" layer="96"/>
 </instance>
-<instance part="R4" gate="G$1" x="71.12" y="10.16" smashed="yes">
-<attribute name="NAME" x="67.31" y="11.6586" size="1.778" layer="95"/>
-<attribute name="VALUE" x="67.31" y="6.858" size="1.778" layer="96"/>
+<instance part="R5" gate="G$1" x="96.52" y="20.32" smashed="yes">
+<attribute name="NAME" x="92.71" y="21.8186" size="1.778" layer="95"/>
+<attribute name="VALUE" x="92.71" y="17.018" size="1.778" layer="96"/>
+</instance>
+<instance part="C1" gate="G$1" x="12.7" y="66.04" smashed="yes" rot="R270">
+<attribute name="NAME" x="13.081" y="64.516" size="1.778" layer="95"/>
+<attribute name="VALUE" x="8.001" y="61.976" size="1.778" layer="96"/>
 </instance>
 </instances>
@@
 </segment>
 <segment>
-<pinref part="R2" gate="G$1" pin="1"/>
 <wire x1="-45.72" y1="33.02" x2="-50.8" y2="33.02" width="0.1524" layer="91"/>
 <label x="-53.34" y="33.02" size="1.778" layer="95"/>
+<pinref part="R2" gate="G$1" pin="1"/>
 </segment>
 <segment>
@@
 </segment>
 <segment>
-<pinref part="R4" gate="G$1" pin="1"/>
 <wire x1="66.04" y1="10.16" x2="60.96" y2="10.16" width="0.1524" layer="91"/>
 <label x="58.42" y="7.62" size="1.778" layer="95"/>
+<pinref part="R3" gate="G$1" pin="1"/>
+</segment>
+<segment>
+<pinref part="C1" gate="G$1" pin="1"/>
+<wire x1="15.24" y1="66.04" x2="17.78" y2="66.04" width="0.1524" layer="91"/>
+<label x="17.78" y="66.04" size="1.778" layer="95"/>
 </segment>
 </net>
@@
 </segment>
 <segment>
-<pinref part="R1" gate="G$1" pin="1"/>
 <wire x1="-30.48" y1="-2.54" x2="-33.02" y2="-2.54" width="0.1524" layer="91"/>
 <wire x1="-33.02" y1="-2.54" x2="-33.02" y2="5.08" width="0.1524" layer="91"/>
@@
 <junction x="-33.02" y="5.08"/>
 <label x="-38.1" y="5.08" size="1.778" layer="95"/>
+<pinref part="R1" gate="G$1" pin="1"/>
 </segment>
 <segment>
@@
 </segment>
 <segment>
-<pinref part="R4" gate="G$1" pin="2"/>
-<pinref part="R3" gate="G$1" pin="1"/>
 <wire x1="76.2" y1="10.16" x2="81.28" y2="10.16" width="0.1524" layer="91"/>
 <wire x1="81.28" y1="10.16" x2="83.82" y2="10.16" width="0.1524" layer="91"/>
@@
 <junction x="81.28" y="10.16"/>
 <label x="81.28" y="-5.08" size="1.778" layer="95"/>
+<pinref part="R3" gate="G$1" pin="2"/>
+<pinref part="R4" gate="G$1" pin="1"/>
 </segment>
 </net>
@@
 <segment>
 <wire x1="101.6" y1="10.16" x2="93.98" y2="10.16" width="0.1524" layer="91"/>
-<pinref part="R3" gate="G$1" pin="2"/>
 <label x="101.6" y="10.16" size="1.778" layer="95"/>
+<pinref part="R4" gate="G$1" pin="2"/>
 </segment>
 </net>
@@
 <net name="N$2" class="0">
 <segment>
-<pinref part="R1" gate="G$1" pin="2"/>
 <pinref part="LD1" gate="G$1" pin="A"/>
 <wire x1="-20.32" y1="-2.54" x2="-17.78" y2="-2.54" width="0.1524" layer="91"/>
+<pinref part="R1" gate="G$1" pin="2"/>
 </segment>
 </net>
 <net name="N$5" class="0">
 <segment>
-<pinref part="R2" gate="G$1" pin="2"/>
 <pinref part="LD2" gate="G$1" pin="C"/>
 <wire x1="-33.02" y1="33.02" x2="-35.56" y2="33.02" width="0.1524" layer="91"/>
+<pinref part="R2" gate="G$1" pin="2"/>
 </segment>
 </net>
@@
 <label x="99.06" y="40.64" size="1.778" layer="95"/>
 </segment>
+<segment>
+<pinref part="R5" gate="G$1" pin="2"/>
+<wire x1="101.6" y1="20.32" x2="104.14" y2="20.32" width="0.1524" layer="91"/>
+<label x="104.14" y="20.32" size="1.778" layer="95"/>
+</segment>
 </net>
 <net name="CANH" class="0">
@@
 <label x="99.06" y="45.72" size="1.778" layer="95"/>
 </segment>
-</net>
+<segment>
+<pinref part="R5" gate="G$1" pin="1"/>
+<wire x1="91.44" y1="20.32" x2="88.9" y2="20.32" width="0.1524" layer="91"/>
+<label x="83.82" y="20.32" size="1.778" layer="95"/>
+</segment>
+</net>
+<net name="EN" class="0">
+<segment>
+<pinref part="U$1" gate="G$1" pin="EN"/>
+<wire x1="-2.54" y1="48.26" x2="-7.62" y2="48.26" width="0.1524" layer="91"/>
+<label x="-10.16" y="48.26" size="1.778" layer="95"/>
+</segment>
+<segment>
+<pinref part="C1" gate="G$1" pin="2"/>
+<wire x1="7.62" y1="66.04" x2="5.08" y2="66.04" width="0.1524" layer="91"/>
+<label x="2.54" y="66.04" size="1.778" layer="95"/>
+</segment>
+</net>
